Commit message: Sensors and Plugins Added

File: urdf/barista_robot_model.urdf (robot description, URDF)
Before this commit: robot barista_bot, 15 links, 14 joints
Links:
- added link laser_scan_frame
- added link laser_scan_link, mass 0.01; collision cylinder length=0.0408 radius=0.037493; visual mesh filename=package://barista_robot_description/meshes/sick_s300.stl scale=0.5 0.5 0.5
- link back_roll_link: geometry collision cylinder length=0.00352 radius=0.025; visual cylinder length=0.00352 radius=0.025
- link back_yaw_link: geometry collision cylinder length=0.00352 radius=0.025; visual cylinder length=0.00352 radius=0.025
- link front_roll_link: geometry collision cylinder length=0.00352 radius=0.025; visual cylinder length=0.00352 radius=0.025
- link front_yaw_link: geometry collision cylinder length=0.00352 radius=0.025; visual cylinder length=0.00352 radius=0.025
Joints:
- added joint laser_scan_frame_joint: type fixed, parent laser_scan_link, child laser_scan_frame, origin xyz=0 0 0.05 rpy=0 0 0, axis 0 0 0
- added joint laser_scan_link_joint: type fixed, parent main_body, child laser_scan_link, origin xyz=0.0 0.0 0.0775 rpy=0 0 0
- joint base_cup_joint: parent base_link -> main_body
- joint left_rod_back_joint: parent base_link -> main_body
- joint left_rod_front_joint: parent base_link -> main_body
- joint right_rod_back_joint: parent base_link -> main_body
- joint right_rod_front_joint: parent base_link -> main_body
