Commit message: Spawning two robots with different namespace

File: xacro/cup_holder_tray.xacro (robot description, xacro)
@@ -17,7 +17,14 @@
                 <cylinder length="${cup_holder_tray_width}" radius="${cup_holder_tray_radius}"/>
                 </geometry>
-                <material name="blue">
-                    <color rgba="0.0 0.0 1.0 1"/>
-                </material>
+                <xacro:if value="${robot_name == 'rick'}">
+                    <material name="blue">
+                        <color rgba="1.0 0.0 0.0 1"/>
+                    </material>
+                </xacro:if>
+                <xacro:if value="${robot_name == 'morty'}">
+                    <material name="red">
+                        <color rgba="0.0 0.0 1.0 1"/>
+                    </material>
+                </xacro:if>
             </visual>
             <collision>
@@ -35,6 +42,11 @@
         </link>
         <gazebo reference="${cup_holder_tray_name}">
-            <material>Gazebo/Blue</material>
-        </gazebo>
+            <xacro:if value="${robot_name == 'rick'}">
+                <material>Gazebo/Blue</material>
+            </xacro:if>
+            <xacro:if value="${robot_name == 'morty'}">
+                <material>Gazebo/Red</material>
+            </xacro:if>
+            </gazebo>
     </xacro:macro>
 </robot>
