Commit message: Robot Stabilized to solve toppling issue

File: xacro/barista_robot_model_rick_morty.urdf.xacro (robot description, xacro)
@@ -23,4 +23,10 @@
         <color rgba="1.0 1.0 1.0 1"/>
     </material>
+    <!-- Macro of cylinder inertia -->
+    <xacro:macro name="cylinder_inertia" params="m r h">
+        <inertia  ixx="${m*(3*r*r+h*h)/12}" ixy = "0" ixz = "0"
+              iyy="${m*(3*r*r+h*h)/12}" iyz = "0"
+              izz="${m*r*r/2}" />
+    </xacro:macro>
     <link name = "base_link">
     </link>
@@ -45,6 +51,7 @@
         <inertial>
             <origin rpy="0 0 0" xyz="0 0 0"/>
-            <mass value="2.0"/>
-            <inertia ixx="0.019846166666666665" ixy="0" ixz="0" iyy="0.019846166666666665" iyz="0" izz="0.031684"/>
+            <mass value="10.0"/>
+             <xacro:cylinder_inertia  m="10.0" r="0.178" h="0.155" />
+            <!-- <inertia ixx="0.019846166666666665" ixy="0" ixz="0" iyy="0.019846166666666665" iyz="0" izz="0.031684"/> -->
         </inertial>
     </link>
@@ -56,4 +63,6 @@
             <material>Gazebo/Red</material>
         </xacro:if>
+        <mu1>0.01</mu1> <!-- Adjust these friction coefficients as needed -->
+        <mu2>0.01</mu2>
     </gazebo>
     <joint name="base_link_joint" type="fixed">
@@ -87,5 +96,5 @@
             <origin rpy="0 1.5707 1.5707" xyz="0 0 0"/>
             <geometry>
-            <cylinder length="0.00352" radius="0.025"/>
+            <cylinder length="0.00352" radius="0.02"/>
             </geometry>
             <material name="blue"/>
@@ -94,5 +103,5 @@
             <origin rpy="0 1.5707 1.5707" xyz="0 0 0"/>
             <geometry>
-            <cylinder length="0.00352" radius="0.025"/>
+            <cylinder length="0.00352" radius="0.02"/>
             </geometry>
         </collision>
@@ -118,5 +127,5 @@
             <origin rpy="0 1.5707 1.5707" xyz="0 0 0"/>
             <geometry>
-            <cylinder length="0.00352" radius="0.025"/>
+            <cylinder length="0.00352" radius="0.02"/>
             </geometry>
             <material name="red"/>
@@ -125,5 +134,5 @@
             <origin rpy="0 1.5707 1.5707" xyz="0 0 0"/>
             <geometry>
-            <cylinder length="0.00352" radius="0.025"/>
+            <cylinder length="0.00352" radius="0.02"/>
             </geometry>
         </collision>
@@ -185,5 +194,5 @@
             <origin rpy="0 1.5707 1.5707" xyz="0 0 0"/>
             <geometry>
-            <cylinder length="0.00352" radius="0.025"/>
+            <cylinder length="0.00352" radius="0.02"/>
             </geometry>
             <material name="blue"/>
@@ -192,5 +201,5 @@
             <origin rpy="0 1.5707 1.5707" xyz="0 0 0"/>
             <geometry>
-            <cylinder length="0.00352" radius="0.025"/>
+            <cylinder length="0.00352" radius="0.02"/>
             </geometry>
         </collision>
@@ -216,5 +225,5 @@
             <origin rpy="0 1.5707 1.5707" xyz="0 0 0"/>
             <geometry>
-            <cylinder length="0.00352" radius="0.025"/>
+            <cylinder length="0.00352" radius="0.02"/>
             </geometry>
             <material name="red"/>
@@ -223,5 +232,5 @@
             <origin rpy="0 1.5707 1.5707" xyz="0 0 0"/>
             <geometry>
-            <cylinder length="0.00352" radius="0.025"/>
+            <cylinder length="0.00352" radius="0.02"/>
             </geometry>
         </collision>

File: xacro/wheel.xacro (robot description, xacro)
@@ -29,12 +29,14 @@
             <inertial>
                 <origin rpy="0 1.5707 1.5707" xyz="0 0 0"/>
-                <mass value="0.75"/>
+                <mass value="3.0"/>
                 <!-- <inertia ixx="0.0002588425" ixy="0" ixz="0" iyy="0.0002588425" iyz="0" izz="0.00046464"/> -->
-                <xacro:cylinder_inertia  m="0.75" r="${wheel_radius}" h="${wheel_width}" />
+                <xacro:cylinder_inertia  m="3.0" r="${wheel_radius}" h="${wheel_width}" />
             </inertial>
         </link>
         <gazebo reference="${wheel_name}">
-            <kp>1000000000000000000000000000.0</kp>
-            <kd>1000000000000000000000000000.0</kd>
+            <!-- <kp>1000000000000000000000000000.0</kp> -->
+            <!-- <kd>1000000000000000000000000000.0</kd> -->
+            <kp>10000000000000.0</kp>
+            <kd>10000000000000.0</kd>
             <mu1>10.0</mu1>
             <mu2>10.0</mu2>
